Commit message: updated include tags in order to follow the new xacro format

File: moveit_manipulation_example/robot_config/urdf/sia20d_workspace.xacro (robot description, xacro)
@@ -1,8 +1,8 @@
 <?xml version="1.0" ?>
 <robot name="sia20d_workspace" xmlns:xacro="http://ros.org/wiki/xacro">
-	<include filename="$(find motoman_config)/cfg/sia20d_mesh_macro.xacro"/>
-	<include filename="$(find robot_config)/urdf/vacuum_gripper_macro.xacro"/>
-	<include filename="$(find robot_config)/urdf/workspace_components.xacro"/>
-	<include filename="$(find robot_config)/urdf/kinect_sensor_macro.xacro"/>
+	<xacro:include filename="$(find motoman_config)/cfg/sia20d_mesh_macro.xacro"/>
+	<xacro:include filename="$(find robot_config)/urdf/vacuum_gripper_macro.xacro"/>
+	<xacro:include filename="$(find robot_config)/urdf/workspace_components.xacro"/>
+	<xacro:include filename="$(find robot_config)/urdf/kinect_sensor_macro.xacro"/>
 	<!-- property list -->
 	<xacro:property name="workcell_height" value="1"/>

File: moveit_manipulation_example/robot_config/urdf/ur5_model.urdf.xacro (robot description, xacro)
@@ -4,5 +4,5 @@
        xmlns:interface="http://playerstage.sourceforge.net/gazebo/xmlschema/#interface"
        xmlns:xacro="http://ros.org/wiki/xacro">
-<include filename="$(find ur5_description)/urdf/arm.transmission.xacro" />
+<xacro:include filename="$(find ur_description)/urdf/ur5.transmission.xacro" />
 <!--
 DH for UR5:
@@ -54,5 +54,5 @@
     <visual>
       <geometry>
-        <mesh filename="package://ur5_description/meshes/Base.dae" />
+        <mesh filename="package://ur_description/meshes/ur5/Base.dae" />
       </geometry>
       <origin xyz="0.0 0.0 0.003" rpy="0.0 0.0 ${3.0 * pi / 4.0}" />
@@ -74,5 +74,5 @@
     <visual>
       <geometry>
-        <mesh filename="package://ur5_description/meshes/Shoulder.dae" />
+        <mesh filename="package://ur_description/meshes/ur5/Shoulder.dae" />
       </geometry>
     </visual>
@@ -100,5 +100,5 @@
     <visual>
       <geometry>
-        <mesh filename="package://ur5_description/meshes/UpperArm.dae" />
+        <mesh filename="package://ur_description/meshes/ur5/UpperArm.dae" />
       </geometry>
       <origin xyz="0.0 0.0 0.0" rpy="0.0 0.0 0.0" />
@@ -127,5 +127,5 @@
     <visual>
       <geometry>
-        <mesh filename="package://ur5_description/meshes/Forearm.dae" />
+        <mesh filename="package://ur_description/meshes/ur5/Forearm.dae" />
       </geometry>
     </visual>
@@ -153,5 +153,5 @@
     <visual>
       <geometry>
-        <mesh filename="package://ur5_description/meshes/Wrist1.dae" />
+        <mesh filename="package://ur_description/meshes/ur5/Wrist1.dae" />
       </geometry>
       <origin xyz="0.0 ${wrist_1_length} 0.0" rpy="0.0 ${pi / 2.0} 0.0" />
@@ -180,5 +180,5 @@
     <visual>
       <geometry>
-        <mesh filename="package://ur5_description/meshes/Wrist2.dae" />
+        <mesh filename="package://ur_description/meshes/ur5/Wrist2.dae" />
       </geometry>
       <origin xyz="0.0 0.0 ${wrist_2_length}" rpy="0.0 0.0 0.0" />
@@ -207,5 +207,5 @@
     <visual>
       <geometry>
-        <mesh filename="package://ur5_description/meshes/Wrist3.dae" />
+        <mesh filename="package://ur_description/meshes/ur5/Wrist3.dae" />
       </geometry>
     </visual>

File: moveit_manipulation_example/robot_config/urdf/ur5_workspace.urdf (robot description, URDF)
Before this commit: robot ur5_workspace, 26 links, 25 joints
Links:
- link base_link: geometry collision mesh filename=package://ur_description/meshes/ur5/collision/Base.dae; visual mesh filename=package://ur_description/meshes/ur5/visual/Base.dae
- link forearm_link: geometry collision mesh filename=package://ur_description/meshes/ur5/collision/Forearm.dae; visual mesh filename=package://ur_description/meshes/ur5/visual/Forearm.dae
- link shoulder_link: geometry collision mesh filename=package://ur_description/meshes/ur5/collision/Shoulder.dae; visual mesh filename=package://ur_description/meshes/ur5/visual/Shoulder.dae
- link upper_arm_link: geometry collision mesh filename=package://ur_description/meshes/ur5/collision/UpperArm.dae; visual mesh filename=package://ur_description/meshes/ur5/visual/UpperArm.dae
- link wrist_1_link: geometry collision mesh filename=package://ur_description/meshes/ur5/collision/Wrist1.dae; visual mesh filename=package://ur_description/meshes/ur5/visual/Wrist1.dae
- link wrist_2_link: geometry collision mesh filename=package://ur_description/meshes/ur5/collision/Wrist2.dae; visual mesh filename=package://ur_description/meshes/ur5/visual/Wrist2.dae
- link wrist_3_link: geometry collision mesh filename=package://ur_description/meshes/ur5/collision/Wrist3.dae; visual mesh filename=package://ur_description/meshes/ur5/visual/Wrist3.dae
Joints:
- joint elbow_joint: axis 0.0 1.0 0.0 -> 0 1 0; limit lower=-0.62831853 upper=2.827433385 effort=10.0 velocity=3.14159265 -> lower=-6.2831853 upper=6.2831853 effort=10.0 velocity=3.14159265
- joint shoulder_lift_joint: axis 0.0 1.0 0.0 -> 0 1 0; limit lower=-3.14159265 upper=3.14159265 effort=10.0 velocity=3.14159265 -> lower=-6.2831853 upper=6.2831853 effort=10.0 velocity=3.14159265
- joint shoulder_pan_joint: axis 0.0 0.0 1.0 -> 0 0 1; limit lower=-2.3561944875 upper=2.3561944875 effort=10.0 velocity=3.14159265 -> lower=-6.2831853 upper=6.2831853 effort=10.0 velocity=3.14159265
- joint wrist_1_joint: axis 0.0 1.0 0.0 -> 0 1 0; limit lower=-3.14159265 upper=0.0314159265 effort=10.0 velocity=3.14159265 -> lower=-3.14159265 upper=0.7853981625 effort=10.0 velocity=3.14159265
- joint wrist_2_joint: axis 0.0 0.0 1.0 -> 0 0 1
- joint wrist_3_joint: axis 0.0 1.0 0.0 -> 0 1 0; limit lower=-4.712388975 upper=4.712388975 effort=10.0 velocity=3.14159265 -> lower=-3.14159265 upper=3.14159265 effort=10.0 velocity=3.14159265

File: moveit_manipulation_example/robot_config/urdf/ur5_workspace.xacro (robot description, xacro)
@@ -1,9 +1,9 @@
 <?xml version="1.0" ?>
 <robot name="ur5_workspace" xmlns:xacro="http://ros.org/wiki/xacro">
-	<include filename="$(find robot_config)/urdf/vacuum_gripper_macro.xacro"/>
-	<include filename="$(find ur5_description)/urdf/gazebo.urdf.xacro" />
-  	<include filename="$(find robot_config)/urdf/ur5_model.urdf.xacro" />
-	<include filename="$(find robot_config)/urdf/workspace_components.xacro"/>
-	<include filename="$(find robot_config)/urdf/kinect_sensor_macro.xacro"/>
+	<xacro:include filename="$(find robot_config)/urdf/vacuum_gripper_macro.xacro"/>
+	<xacro:include filename="$(find ur_description)/urdf/gazebo.urdf.xacro" />
+  	<xacro:include filename="$(find ur_description)/urdf/ur5.urdf.xacro" />
+	<xacro:include filename="$(find robot_config)/urdf/workspace_components.xacro"/>
+	<xacro:include filename="$(find robot_config)/urdf/kinect_sensor_macro.xacro"/>
 	<!-- property list -->
 	<xacro:property name="workcell_height" value="1"/>
